File: fpga/bay/card/omnimeter-card.kicad_sch (KiCad schematic)
At the start: 0 parts

Commit message: handoff
Other:
- added sheet Config (config.kicad_sch)
- added sheet Core power (core_power.kicad_sch)
- added sheet FPGA (fpga.kicad_sch)
- added sheet Fan pass-through (fan.kicad_sch)
- added sheet Interposer (interposer.kicad_sch)
- added sheet Management (mgmt.kicad_sch)
- added sheet PCIe sideband (pcie_sideband.kicad_sch)
- added sheet Power input (power_in.kicad_sch)
Changed lines of the file:
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@@
 	(generator_version "10.0")
 	(paper "A4")
+  (sheet
+    (at 25.4 30.48)
+    (size 50.8 25.4)
+    (exclude_from_sim no)
+    (in_bom yes)
+    (on_board yes)
+    (dnp no)
+    (fields_autoplaced yes)
+    (stroke (width 0.1524) (type solid))
+    (fill (color 0 0 0 0.0))
+    (property "Sheetname" "Interposer"
+      (at 25.4 29.845 0)
+      (show_name no)
+      (do_not_autoplace no)
+      (effects (font (size 1.27 1.27)) (justify left bottom))
+    )
+    (property "Sheetfile" "interposer.kicad_sch"
+      (at 25.4 56.51499999999999 0)
+      (show_name no)
+      (do_not_autoplace no)
+      (effects (font (size 1.27 1.27)) (justify left top))
+    )
+    (instances
+      (project "omnimeter-card"
+        (path "/d7dcd351-036e-417b-86ff-4ba43184a562" (page "2"))
+      )
+    )
+  )
+  (sheet
+    (at 91.44 30.48)
+    (size 50.8 25.4)
+    (exclude_from_sim no)
+    (in_bom yes)
+    (on_board yes)
+    (dnp no)
+    (fields_autoplaced yes)
+    (stroke (width 0.1524) (type solid))
+    (fill (color 0 0 0 0.0))
+    (property "Sheetname" "Fan pass-through"
+      (at 91.44 29.845 0)
+      (show_name no)
+      (do_not_autoplace no)
+      (effects (font (size 1.27 1.27)) (justify left bottom))
+    )
+    (property "Sheetfile" "fan.kicad_sch"
+      (at 91.44 56.51499999999999 0)
+      (show_name no)
+      (do_not_autoplace no)
+      (effects (font (size 1.27 1.27)) (justify left top))
+    )
+    (instances
+      (project "omnimeter-card"
+        (path "/d7dcd351-036e-417b-86ff-4ba43184a562" (page "3"))
+      )
+    )
+  )
+  (sheet
+    (at 157.48 30.48)
+    (size 50.8 25.4)
+    (exclude_from_sim no)
+    (in_bom yes)
+    (on_board yes)
+    (dnp no)
+    (fields_autoplaced yes)
+    (stroke (width 0.1524) (type solid))
+    (fill (color 0 0 0 0.0))
+    (property "Sheetname" "Management"
+      (at 157.48 29.845 0)
+      (show_name no)
+      (do_not_autoplace no)
+      (effects (font (size 1.27 1.27)) (justify left bottom))
+    )
+    (property "Sheetfile" "mgmt.kicad_sch"
+      (at 157.48 56.51499999999999 0)
+      (show_name no)
+      (do_not_autoplace no)
+      (effects (font (size 1.27 1.27)) (justify left top))
+    )
+    (instances
+      (project "omnimeter-card"
+        (path "/d7dcd351-036e-417b-86ff-4ba43184a562" (page "4"))
+      )
+    )
+  )
+  (sheet
+    (at 25.4 76.2)
+    (size 50.8 25.4)
+    (exclude_from_sim no)
+    (in_bom yes)
+    (on_board yes)
+    (dnp no)
+    (fields_autoplaced yes)
+    (stroke (width 0.1524) (type solid))
+    (fill (color 0 0 0 0.0))
+    (property "Sheetname" "Power input"
+      (at 25.4 75.565 0)
+      (show_name no)
+      (do_not_autoplace no)
+      (effects (font (size 1.27 1.27)) (justify left bottom))
+    )
+    (property "Sheetfile" "power_in.kicad_sch"
+      (at 25.4 102.235 0)
+      (show_name no)
+      (do_not_autoplace no)
+      (effects (font (size 1.27 1.27)) (justify left top))
+    )
+    (instances
+      (project "omnimeter-card"
+        (path "/d7dcd351-036e-417b-86ff-4ba43184a562" (page "5"))
+      )
+    )
+  )
+  (sheet
+    (at 91.44 76.2)
+    (size 50.8 25.4)
+    (exclude_from_sim no)
+    (in_bom yes)
+    (on_board yes)
+    (dnp no)
+    (fields_autoplaced yes)
+    (stroke (width 0.1524) (type solid))
+    (fill (color 0 0 0 0.0))
+    (property "Sheetname" "Core power"
+      (at 91.44 75.565 0)
+      (show_name no)
+      (do_not_autoplace no)
+      (effects (font (size 1.27 1.27)) (justify left bottom))
+    )
+    (property "Sheetfile" "core_power.kicad_sch"
+      (at 91.44 102.235 0)
+      (show_name no)
+      (do_not_autoplace no)
+      (effects (font (size 1.27 1.27)) (justify left top))
+    )
+    (instances
+      (project "omnimeter-card"
+        (path "/d7dcd351-036e-417b-86ff-4ba43184a562" (page "6"))
+      )
+    )
+  )
+  (sheet
+    (at 157.48 76.2)
+    (size 50.8 25.4)
+    (exclude_from_sim no)
+    (in_bom yes)
+    (on_board yes)
+    (dnp no)
+    (fields_autoplaced yes)
+    (stroke (width 0.1524) (type solid))
+    (fill (color 0 0 0 0.0))
+    (property "Sheetname" "PCIe sideband"
+      (at 157.48 75.565 0)
+      (show_name no)
+      (do_not_autoplace no)
+      (effects (font (size 1.27 1.27)) (justify left bottom))
+    )
+    (property "Sheetfile" "pcie_sideband.kicad_sch"
+      (at 157.48 102.235 0)
+      (show_name no)
+      (do_not_autoplace no)
+      (effects (font (size 1.27 1.27)) (justify left top))
+    )
+    (instances
+      (project "omnimeter-card"
+        (path "/d7dcd351-036e-417b-86ff-4ba43184a562" (page "7"))
+      )
+    )
+  )
+  (sheet
+    (at 25.4 121.92)
+    (size 50.8 25.4)
+    (exclude_from_sim no)
+    (in_bom yes)
+    (on_board yes)
+    (dnp no)
+    (fields_autoplaced yes)
+    (stroke (width 0.1524) (type solid))
+    (fill (color 0 0 0 0.0))
+    (property "Sheetname" "Config"
+      (at 25.4 121.285 0)
+      (show_name no)
+      (do_not_autoplace no)
+      (effects (font (size 1.27 1.27)) (justify left bottom))
+    )
+    (property "Sheetfile" "config.kicad_sch"
+      (at 25.4 147.95499999999998 0)
+      (show_name no)
+      (do_not_autoplace no)
+      (effects (font (size 1.27 1.27)) (justify left top))
+    )
+    (instances
+      (project "omnimeter-card"
+        (path "/d7dcd351-036e-417b-86ff-4ba43184a562" (page "8"))
+      )
+    )
+  )
+  (sheet
+    (at 91.44 121.92)
+    (size 50.8 25.4)
+    (exclude_from_sim no)
+    (in_bom yes)
+    (on_board yes)
+    (dnp no)
+    (fields_autoplaced yes)
+    (stroke (width 0.1524) (type solid))
+    (fill (color 0 0 0 0.0))
+    (property "Sheetname" "FPGA"
+      (at 91.44 121.285 0)
+      (show_name no)
+      (do_not_autoplace no)
+      (effects (font (size 1.27 1.27)) (justify left bottom))
+    )
+    (property "Sheetfile" "fpga.kicad_sch"
+      (at 91.44 147.95499999999998 0)
+      (show_name no)
+      (do_not_autoplace no)
+      (effects (font (size 1.27 1.27)) (justify left top))
+    )
+    (instances
+      (project "omnimeter-card"
+        (path "/d7dcd351-036e-417b-86ff-4ba43184a562" (page "9"))
+      )
+    )
+  )
+  (sheet_instances
+    (path "/"
+      (page "1")
+    )
+  )
+  (embedded_fonts no)
 )
