File: fpga/bay/card/fan.kicad_sch (KiCad schematic)
At the start: 0 parts

Commit message: Phase 2 path2: fan + mgmt sheets (AFC58 connectors, 24LC32 EEPROM @0x50, test pads)
Co-Authored-By: Claude Opus 5.5 <noreply@anthropic.com>
Parts:
- added C1: 10u/25V, Capacitor_SMD:C_1206_3216Metric, symbol Device:C
- added J2, J3: AFC58-S04FIA-R1, symbol Connector_Generic:Conn_01x04
Connections:
- new net +12V_FAN: C1.1, J2.1 (Pin_1), J3.1 (Pin_1)
- new net FAN0_PWM: J2.3 (Pin_3)
- new net FAN0_SPEED: J2.2 (Pin_2)
- new net FAN1_PWM: J3.3 (Pin_3)
- new net FAN1_SPEED: J3.2 (Pin_2)
- new net GND: C1.2, J2.4 (Pin_4), J3.4 (Pin_4)

Commit message: Phase 2 path2: AFC58-S04FIA-R1 footprint, assigned to J2/J3; verified land pattern note
Co-Authored-By: Claude Opus 5.5 <noreply@anthropic.com>
Parts:
- J2, J3: footprint (none) -> omnimeter:AFC58-S04FIA-R1
Changed lines of the file:
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@@
 			)
 		)
-		(property "Footprint" ""
+		(property "Footprint" "omnimeter:AFC58-S04FIA-R1"
 			(at 127 88.9 0)
 			(hide yes)
@@
 			)
 		)
-		(property "Footprint" ""
+		(property "Footprint" "omnimeter:AFC58-S04FIA-R1"
 			(at 127 139.7 0)
 			(hide yes)

Commit message: fpga: rename KiCad project and library omnimeter-card/omnimeter -> fw16-fpga-module
Co-Authored-By: Claude Opus 5.5 (1M context) <noreply@anthropic.com>
Claude-Session: https://claude.ai/code/session_019QA2U79cSHCaAaMe6Km575
Parts:
- J2, J3: footprint omnimeter:AFC58-S04FIA-R1 -> fw16-fpga-module:AFC58-S04FIA-R1
Changed lines of the file:
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@@
 			)
 		)
-		(property "Footprint" "omnimeter:AFC58-S04FIA-R1"
+		(property "Footprint" "fw16-fpga-module:AFC58-S04FIA-R1"
 			(at 127 88.9 0)
 			(hide yes)
@@
 		)
 		(instances
-			(project "omnimeter-card"
+			(project "fw16-fpga-module"
 				(path "/d7dcd351-036e-417b-86ff-4ba43184a562/77c85ed9-b6df-4ddd-ab26-1cbdf63af543"
 					(reference "J2")
@@
 			)
 		)
-		(property "Footprint" "omnimeter:AFC58-S04FIA-R1"
+		(property "Footprint" "fw16-fpga-module:AFC58-S04FIA-R1"
 			(at 127 139.7 0)
 			(hide yes)
@@
 		)
 		(instances
-			(project "omnimeter-card"
+			(project "fw16-fpga-module"
 				(path "/d7dcd351-036e-417b-86ff-4ba43184a562/77c85ed9-b6df-4ddd-ab26-1cbdf63af543"
 					(reference "J3")
@@
 		)
 		(instances
-			(project "omnimeter-card"
+			(project "fw16-fpga-module"
 				(path "/d7dcd351-036e-417b-86ff-4ba43184a562/77c85ed9-b6df-4ddd-ab26-1cbdf63af543"
 					(reference "C1")
@@
 		)
 		(instances
-			(project "omnimeter-card"
+			(project "fw16-fpga-module"
 				(path "/d7dcd351-036e-417b-86ff-4ba43184a562/77c85ed9-b6df-4ddd-ab26-1cbdf63af543"
 					(reference "#PWR01")
@@
 		)
 		(instances
-			(project "omnimeter-card"
+			(project "fw16-fpga-module"
 				(path "/d7dcd351-036e-417b-86ff-4ba43184a562/77c85ed9-b6df-4ddd-ab26-1cbdf63af543"
 					(reference "#PWR02")
@@
 		)
 		(instances
-			(project "omnimeter-card"
+			(project "fw16-fpga-module"
 				(path "/d7dcd351-036e-417b-86ff-4ba43184a562/77c85ed9-b6df-4ddd-ab26-1cbdf63af543"
 					(reference "#PWR03")
