File: fpga/bay/card/mgmt.kicad_sch (KiCad schematic)
At the start: 0 parts

Commit message: Phase 2 path2: fan + mgmt sheets (AFC58 connectors, 24LC32 EEPROM @0x50, test pads)
Co-Authored-By: Claude Opus 5.5 <noreply@anthropic.com>
Parts:
- added C2: 100n, Capacitor_SMD:C_0402_1005Metric, symbol Device:C
- added JP1: WP_EN, Jumper:SolderJumper-2_P1.3mm_Open_Pad1.0x1.5mm, symbol Jumper:SolderJumper_2_Open
- added R3: 10k, Resistor_SMD:R_0402_1005Metric, symbol Device:R
- added R4, R5: 2.2k DNP, Resistor_SMD:R_0402_1005Metric, symbol Device:R
- added TP1: VSYS_GPU, TestPoint:TestPoint_Pad_D1.0mm, symbol Connector:TestPoint
- added TP10: TH_ALERT#, TestPoint:TestPoint_Pad_D1.0mm, symbol Connector:TestPoint
- added TP11: TH_OVERT#, TestPoint:TestPoint_Pad_D1.0mm, symbol Connector:TestPoint
- added TP12: I2C_ALW_INT, TestPoint:TestPoint_Pad_D1.0mm, symbol Connector:TestPoint
- added TP13: GPIO0_EC, TestPoint:TestPoint_Pad_D1.0mm, symbol Connector:TestPoint
- added TP14: GPIO1_EC, TestPoint:TestPoint_Pad_D1.0mm, symbol Connector:TestPoint
- added TP15: GPIO2_EC, TestPoint:TestPoint_Pad_D1.0mm, symbol Connector:TestPoint
- added TP16: GPIO3_EC, TestPoint:TestPoint_Pad_D1.0mm, symbol Connector:TestPoint
- added TP17: USB_P, TestPoint:TestPoint_Pad_D1.0mm, symbol Connector:TestPoint
- added TP18: USB_N, TestPoint:TestPoint_Pad_D1.0mm, symbol Connector:TestPoint
- added TP19: DP_A_AUX, TestPoint:TestPoint_Pad_D1.0mm, symbol Connector:TestPoint
- added TP2: +5V_ALW, TestPoint:TestPoint_Pad_D1.0mm, symbol Connector:TestPoint
- added TP20: DP_A_AUX#, TestPoint:TestPoint_Pad_D1.0mm, symbol Connector:TestPoint
- added TP21: EXT_SSD1_RST#, TestPoint:TestPoint_Pad_D1.0mm, symbol Connector:TestPoint
- added TP22: EXT_SSD2_RST#, TestPoint:TestPoint_Pad_D1.0mm, symbol Connector:TestPoint
- added TP23: EXT_SSD2_CLKREQ#, TestPoint:TestPoint_Pad_D1.0mm, symbol Connector:TestPoint
- added TP3: +3V3_ALW, TestPoint:TestPoint_Pad_D1.0mm, symbol Connector:TestPoint
- added TP4: +12V_FAN, TestPoint:TestPoint_Pad_D1.0mm, symbol Connector:TestPoint
- added TP5: GND, TestPoint:TestPoint_Pad_D1.0mm, symbol Connector:TestPoint
- added TP6: PWR_EN, TestPoint:TestPoint_Pad_D1.0mm, symbol Connector:TestPoint
- added TP7: PWR_GOOD, TestPoint:TestPoint_Pad_D1.0mm, symbol Connector:TestPoint
- added TP8: PEX_RST#, TestPoint:TestPoint_Pad_D1.0mm, symbol Connector:TestPoint
- added TP9: PEX_CLKREQ#, TestPoint:TestPoint_Pad_D1.0mm, symbol Connector:TestPoint
- added U1: 24LC32, Package_SO:TSSOP-8_4.4x3mm_P0.65mm, symbol Memory_EEPROM:24LC32
Connections:
- new net: JP1.1 (A), R3.1, U1.7 (WP)
- new net +12V_FAN: TP4.1
- new net +3V3_ALW: C2.1, JP1.2 (B), R4.1, R5.1, TP3.1, U1.8 (VCC)
- new net +5V_ALW: TP2.1
- new net DP_A_AUX: TP19.1
- new net DP_A_AUX#: TP20.1
- new net EXT_SSD1_RST#: TP21.1
- new net EXT_SSD2_CLKREQ#: TP23.1
- new net EXT_SSD2_RST#: TP22.1
- new net GND: C2.2, R3.2, TP5.1, U1.1 (A0), U1.2 (A1), U1.3 (A2), U1.4 (GND)
- new net GPIO0_EC: TP13.1
- new net GPIO1_EC: TP14.1
- new net GPIO2_EC: TP15.1
- new net GPIO3_EC: TP16.1
- new net I2C_ALW_INT: TP12.1
- new net I2C_ALW_SCL: R4.2, U1.6 (SCL)
- new net I2C_ALW_SDA: R5.2, U1.5 (SDA)
- new net PEX_CLKREQ#: TP9.1
- new net PEX_RST#: TP8.1
- new net PWR_EN: TP6.1
- new net PWR_GOOD: TP7.1
- new net TH_ALERT#: TP10.1
- new net TH_OVERT#: TP11.1
- new net USB_N: TP18.1
- new net USB_P: TP17.1
- new net VSYS_GPU: TP1.1
