File: fpga/bay/card/power_in.kicad_sch (KiCad schematic)
At the start: 0 parts

Commit message: Phase 2 path2: power_in sheet (TPS259474L eFuse, INA237 monitor, LMR33630 5V0 buck) + RPW0010A footprint/symbol
Co-Authored-By: Claude Opus 5.5 <noreply@anthropic.com>
Parts:
- added C10, C7, C9: 10u/25V, Capacitor_SMD:C_1206_3216Metric, symbol Device:C
- added C11, C4: 100n/25V, Capacitor_SMD:C_0402_1005Metric, symbol Device:C
- added C12, C8: 100n, Capacitor_SMD:C_0402_1005Metric, symbol Device:C
- added C13: 1u, Capacitor_SMD:C_0402_1005Metric, symbol Device:C
- added C14, C15, C16: 22u/16V, Capacitor_SMD:C_1206_3216Metric, symbol Device:C
- added C3: 1u/25V, Capacitor_SMD:C_0603_1608Metric, symbol Device:C
- added C5: 10n, Capacitor_SMD:C_0402_1005Metric, symbol Device:C
- added C6: 2.2n, Capacitor_SMD:C_0402_1005Metric, symbol Device:C
- added L1: 10u XAL5030-103, Inductor_SMD:L_Coilcraft_XAL5030-XXX, symbol Device:L
- added R10: 1.33k, Resistor_SMD:R_0402_1005Metric, symbol Device:R
- added R11, R6: 390k, Resistor_SMD:R_0402_1005Metric, symbol Device:R
- added R12, R7: 91k, Resistor_SMD:R_0402_1005Metric, symbol Device:R
- added R13, R17, R20: 10k, Resistor_SMD:R_0402_1005Metric, symbol Device:R
- added R14: 10m 1%, Resistor_SMD:R_1206_3216Metric, symbol Device:R
- added R15, R16: 4.7k, Resistor_SMD:R_0402_1005Metric, symbol Device:R
- added R18: 100k, Resistor_SMD:R_0402_1005Metric, symbol Device:R
- added R19: 24.9k, Resistor_SMD:R_0402_1005Metric, symbol Device:R
- added R8: 1M, Resistor_SMD:R_0402_1005Metric, symbol Device:R
- added R9: 57.6k, Resistor_SMD:R_0402_1005Metric, symbol Device:R
- added U2: TPS259474LRPW, omnimeter:Texas_RPW0010A_VQFN-HR-10_2x2mm, symbol omnimeter:TPS259474LRPW
- added U3: INA237AIDGSR, Package_SO:TSSOP-10_3x3mm_P0.5mm, symbol Sensor_Energy:INA237
- added U4: LMR33630ADDA, Package_SO:Texas_HSOP-8-1EP_3.9x4.9mm_P1.27mm_ThermalVias, symbol Regulator_Switching:LMR33630ADDA
Connections:
- new net +3V3_ALW: C8.1, R13.1, R15.1, R16.1, R17.1, R20.1, U3.6 (VS)
- new net +5V0_MAIN: C14.1, C15.1, C16.1, L1.2, R18.1
- new net 5V0_PG: R20.2, U4.4 (PG)
- new net BUCK_BOOT: C12.1, U4.7 (BOOT)
- new net BUCK_FB: R18.2, R19.1, U4.5 (FB)
- new net BUCK_SW: C12.2, L1.1, U4.8 (SW)
- new net BUCK_VCC: C13.1, U4.6 (VCC)
- new net EFUSE_DVDT: C5.1, U2.7 (DVDT)
- new net EFUSE_EN: R6.2, R7.1, U2.1 (EN/UVLO)
- new net EFUSE_ILM: R10.1, U2.9 (ILM)
- new net EFUSE_ITIMER: C6.1, U2.10 (ITIMER)
- new net EFUSE_OVLO: R8.2, R9.1, U2.2 (OVLO)
- new net EFUSE_PGTH: R11.2, R12.1, U2.4 (PGTH)
- new net GND: C10.2, C11.2, C13.2, C14.2, C15.2, C16.2, C3.2, C4.2, C5.2, C6.2, C7.2, C8.2, C9.2, R10.2, R12.2, R19.2, R7.2, R9.2, U2.8 (GND), U3.1 (A1), U3.2 (A0), U3.7 (GND), U4.1 (GND), U4.9 (GND)
- new net SENSE_ALERT#: R17.2, U3.3 (~{Alert})
- new net SENSE_SCL: R15.2, U3.5 (SCL)
- new net SENSE_SDA: R16.2, U3.4 (SDA)
- new net VSYS_F: C7.1, R11.1, R14.1, U2.6 (OUT), U3.10 (Vin+)
- new net VSYS_GPU: C3.1, C4.1, R6.1, R8.1, U2.5 (IN)
- new net VSYS_PG: R13.2, U2.3 (PG), U4.3 (EN)
- new net VSYS_SNS: C10.1, C11.1, C9.1, R14.2, U3.8 (Vbus), U3.9 (Vin-), U4.2 (VIN)

Commit message: Phase 2: sense-bus pull-ups to +3V3_IO; worker logs/lessons (2b, 3c); path3 handoff step-4 note
Co-Authored-By: Claude Opus 5.5 <noreply@anthropic.com>
Connections:
- net +3V3_ALW: no longer R15.1, R16.1, R17.1
- new net +3V3_IO: R15.1, R16.1, R17.1
Changed lines of the file:
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@@
-	(global_label "+3V3_ALW"
-		(shape input)
-		(at 35.56 146.05 0)
-		(effects
-			(font
-				(size 1.27 1.27)
-			)
-			(justify left)
-		)
-	)
-	(global_label "+3V3_ALW"
-		(shape input)
-		(at 50.8 146.05 0)
-		(effects
-			(font
-				(size 1.27 1.27)
-			)
-			(justify left)
-		)
-	)
-	(global_label "+3V3_ALW"
-		(shape input)
-		(at 66.04 146.05 0)
-		(effects
-			(font
-				(size 1.27 1.27)
-			)
-			(justify left)
-		)
-	)
 	(global_label "+3V3_ALW"
 		(shape input)
@@
 		(effects
 			(font
+				(size 1.27 1.27)
+			)
+			(justify left)
+		)
+	)
+	(global_label "+3V3_IO"
+		(shape input)
+		(at 35.56 146.05 0)
+		(effects
+			(font
+				(size 1.27 1.27)
+			)
+			(justify left)
+		)
+	)
+	(global_label "+3V3_IO"
+		(shape input)
+		(at 50.8 146.05 0)
+		(effects
+			(font
+				(size 1.27 1.27)
+			)
+			(justify left)
+		)
+	)
+	(global_label "+3V3_IO"
+		(shape input)
+		(at 66.04 146.05 0)
+		(effects
+			(font

Commit message: fpga: rename KiCad project and library omnimeter-card/omnimeter -> fw16-fpga-module
Co-Authored-By: Claude Opus 5.5 (1M context) <noreply@anthropic.com>
Claude-Session: https://claude.ai/code/session_019QA2U79cSHCaAaMe6Km575
Parts:
- U2: footprint omnimeter:Texas_RPW0010A_VQFN-HR-10_2x2mm -> fw16-fpga-module:Texas_RPW0010A_VQFN-HR-10_2x2mm; symbol omnimeter:TPS259474LRPW -> fw16-fpga-module:TPS259474LRPW
