File: fpga/bay/card/pcie_sideband.kicad_sch (KiCad schematic)
At the start: 0 parts

Commit message: card: pcie_sideband sheet (TH_* open-drain 2N7002K, CLKREQ# 0R strap + DNP to FPGA) per decision 0010
Co-Authored-By: Claude Opus 5.5 (1M context) <noreply@anthropic.com>
Claude-Session: https://claude.ai/code/session_019QA2U79cSHCaAaMe6Km575
Parts:
- added Q1, Q2: 2N7002K, Package_TO_SOT_SMD:SOT-23, symbol Transistor_FET:2N7002K
- added R21, R22: 100k, Resistor_SMD:R_0402_1005Metric, symbol Device:R
- added R23: 0R, Resistor_SMD:R_0402_1005Metric, symbol Device:R
- added R24: 0R DNP, Resistor_SMD:R_0402_1005Metric, symbol Device:R
Connections:
- new net FPGA_CLKREQ_N: R24.2
- new net FPGA_TH_ALERT: Q1.1 (G), R21.1
- new net FPGA_TH_OVERT: Q2.1 (G), R22.1
- new net GND: Q1.2 (S), Q2.2 (S), R21.2, R22.2, R23.2
- new net PEX_CLKREQ#: R23.1, R24.1
- new net TH_ALERT#: Q1.3 (D)
- new net TH_OVERT#: Q2.3 (D)
