File: fpga/bay/card/config.kicad_sch (KiCad schematic)
At the start: 0 parts

Commit message: card: config sheet (MT25QU256 x4 QSPI, UG570 pull-ups/straps, TC2050 Xilinx JTAG) per decision 0010
Co-Authored-By: Claude Opus 5.5 (1M context) <noreply@anthropic.com>
Claude-Session: https://claude.ai/code/session_019QA2U79cSHCaAaMe6Km575
Parts:
- added C17: 100n, Capacitor_SMD:C_0402_1005Metric, symbol Device:C
- added J4: TC2050-IDC-NL (Xilinx), Connector:Tag-Connect_TC2050-IDC-NL_2x05_P1.27mm_Vertical, symbol Connector_Generic:Conn_02x05_Odd_Even
- added R25: 2.4k, Resistor_SMD:R_0402_1005Metric, symbol Device:R
- added R26, R27, R28, R29, R30: 4.7k, Resistor_SMD:R_0402_1005Metric, symbol Device:R
- added R31, R32, R33, R34: 1k, Resistor_SMD:R_0402_1005Metric, symbol Device:R
- added U5: MT25QU256ABA1EW7, Package_DFN_QFN:W-PDFN-8-1EP_6x5mm_P1.27mm_EP3x3mm, symbol Memory_Flash:MT25QUxxxxxx1xW7
Connections:
- new net +1V8: C17.1, J4.1 (Pin_1), R25.1, R26.1, R27.1, R28.1, R29.1, R30.1, R31.1, R34.1, U5.8 (VCC)
- new net FPGA_CCLK: U5.6 (C)
- new net FPGA_D00: U5.5 (DQ0)
- new net FPGA_D01: U5.2 (DQ1)
- new net FPGA_D02: R26.2, U5.3 (~{W}/DQ2)
- new net FPGA_D03: R27.2, U5.7 (~{RESET}/DQ3)
- new net FPGA_DONE: R30.2
- new net FPGA_FCS_B: R25.2, U5.1 (~{S})
- new net FPGA_INIT_B: R29.2
- new net FPGA_M0: R31.2
- new net FPGA_M1: R32.1
- new net FPGA_M2: R33.1
- new net FPGA_PROGRAM_B: R28.2
- new net FPGA_PUDC_B: R34.2
- new net FPGA_TCK: J4.4 (Pin_4)
- new net FPGA_TDI: J4.8 (Pin_8)
- new net FPGA_TDO: J4.6 (Pin_6)
- new net FPGA_TMS: J4.2 (Pin_2)
- new net GND: C17.2, J4.3 (Pin_3), J4.5 (Pin_5), J4.7 (Pin_7), J4.9 (Pin_9), R32.2, R33.2, U5.4 (VSS), U5.9 (PAD)
- no-connect marks 0 -> 1
