File: fpga/bay/card/core_power.kicad_sch (KiCad schematic)
At the start: 0 parts

Commit message: card: core_power sheet (LM3880 sequencer, TPS566238P VCCINT, TLV62569P 1V8/1V6, TPS7A84A MGT LDOs, TLV755 aux/3V3_IO); netlist identical to omnimeter 0ee72b0
Co-Authored-By: Claude Opus 5.5 (1M context) <noreply@anthropic.com>
Claude-Session: https://claude.ai/code/session_019QA2U79cSHCaAaMe6Km575
Parts:
- added C18, C21, C22: 100n, Capacitor_SMD:C_0402_1005Metric, symbol Device:C
- added C19, C20, C28, C30, C36, C41: 10u/10V, Capacitor_SMD:C_0805_2012Metric, symbol Device:C
- added C23, C33, C35: 1u, Capacitor_SMD:C_0402_1005Metric, symbol Device:C
- added C24, C25, C26, C27, C29, C31: 22u/6.3V, Capacitor_SMD:C_0805_2012Metric, symbol Device:C
- added C32, C34, C37, C42: 1u/10V, Capacitor_SMD:C_0402_1005Metric, symbol Device:C
- added C38, C43: 10n, Capacitor_SMD:C_0402_1005Metric, symbol Device:C
- added C39, C44: 47u/6.3V, Capacitor_SMD:C_1206_3216Metric, symbol Device:C
- added C40, C45: 10u/6.3V, Capacitor_SMD:C_0805_2012Metric, symbol Device:C
- added L2: 1u XAL4020-102, Inductor_SMD:L_Coilcraft_XAL4020-XXX, symbol Device:L
- added L3, L4: 2.2u DFE201610, Inductor_SMD:L_Murata_DFE201610P, symbol Device:L
- added R35, R36, R37, R40, R42, R43, R46, R47: 100k, Resistor_SMD:R_0402_1005Metric, symbol Device:R
- added R38: 8.45k 0.1%, Resistor_SMD:R_0402_1005Metric, symbol Device:R
- added R39: 20k 0.1%, Resistor_SMD:R_0402_1005Metric, symbol Device:R
- added R41, R44: 200k, Resistor_SMD:R_0402_1005Metric, symbol Device:R
- added R45: 120k, Resistor_SMD:R_0402_1005Metric, symbol Device:R
- added U10: TLV75518PDBV, Package_TO_SOT_SMD:SOT-23-5, symbol Regulator_Linear:TLV75518PDBV
- added U11: TLV75533PDBV, Package_TO_SOT_SMD:SOT-23-5, symbol Regulator_Linear:TLV75533PDBV
- added U12, U13: TPS7A8400ARGR, Package_DFN_QFN:QFN-20-1EP_3.5x3.5mm_P0.5mm_EP2x2mm_ThermalVias, symbol fw16-fpga-module:TPS7A8400ARGR
- added U6: LM3880MF-1AE, Package_TO_SOT_SMD:SOT-23-6, symbol Power_Supervisor:LM3880
- added U7: TPS566238PRQF, fw16-fpga-module:Texas_RQF0009A_VQFN-HR-9_1.5x2mm, symbol fw16-fpga-module:TPS566238PRQF
- added U8, U9: TLV62569PDRL, Package_TO_SOT_SMD:SOT-563, symbol fw16-fpga-module:TLV62569PDRL
Connections:
- new net +0V85_VCCINT: C24.1, C25.1, C26.1, C27.1, L2.2, R38.1
- new net +0V9_MGTAVCC: C39.1, C40.1, U12.1 (OUT), U12.19 (OUT), U12.2 (SNS), U12.20 (OUT)
- new net +1V2_MGTAVTT: C44.1, C45.1, U13.1 (OUT), U13.19 (OUT), U13.2 (SNS), U13.20 (OUT)
- new net +1V6_MGT: C31.1, C36.1, C41.1, L4.2, R44.1, U12.15 (IN), U12.16 (IN), U12.17 (IN), U13.15 (IN), U13.16 (IN), U13.17 (IN)
- new net +1V8: C29.1, L3.2, R41.1
- new net +1V8_MGTVCCAUX: C33.1, U10.5 (OUT)
- new net +3V3_ALW: R40.1, R43.1, R47.1
- new net +3V3_IO: C35.1, U11.5 (OUT)
- new net +5V0_MAIN: C18.1, C19.1, C20.1, C21.1, C28.1, C30.1, C32.1, C34.1, C37.1, C42.1, R35.1, R36.1, R37.1, R46.1, U10.1 (IN), U10.3 (EN), U11.1 (IN), U12.12 (BIAS), U13.12 (BIAS), U6.1 (VCC), U7.5 (VIN), U7.6 (VIN), U8.3 (VIN), U9.3 (VIN)
- new net 1V6_FB: R44.2, R45.1, U9.1 (FB)
- new net 1V6_SW: L4.1, U9.4 (SW)
- new net 1V8_FB: R41.2, R42.1, U8.1 (FB)
- new net 1V8_SW: L3.1, U8.4 (SW)
- new net 5V0_PG: U6.3 (EN)
- new net EN_AUX: R36.2, U6.5 (FLAG2), U8.5 (EN), U9.5 (EN)
- new net EN_MGT: R37.2, U11.3 (EN), U12.14 (EN), U6.4 (FLAG3)
- new net EN_VCCINT: R35.2, U6.6 (FLAG1), U7.3 (EN)
- new net GND: C18.2, C19.2, C20.2, C21.2, C23.2, C24.2, C25.2, C26.2, C27.2, C28.2, C29.2, C30.2, C31.2, C32.2, C33.2, C34.2, C35.2, C36.2, C37.2, C38.2, C39.2, C40.2, C41.2, C42.2, C43.2, C44.2, C45.2, R39.2, R42.2, R45.2, U10.2 (GND), U11.2 (GND), U12.18 (GND), U12.21 (EP), U12.6 (100mV), U12.8 (GND), U13.18 (GND), U13.21 (EP), U13.8 (GND), U13.9 (400mV), U6.2 (GND), U7.4 (PGND), U8.2 (GND), U9.2 (GND)
- new net MGTAVCC_NR: C38.1, U12.13 (NR/SS)
- new net MGTAVCC_PG: R46.2, U12.4 (PG), U13.14 (EN)
- new net MGTAVTT_NR: C43.1, U13.13 (NR/SS)
- new net MGTAVTT_PG: R47.2, U13.4 (PG)
- new net VCC1V8_PG: R43.2, U8.6 (PG)
- new net VCCINT_BST: C22.1, U7.7 (BST)
- new net VCCINT_FB: R38.2, R39.1, U7.2 (FB)
- new net VCCINT_PG: R40.2, U7.9 (PG)
- new net VCCINT_SW: C22.2, L2.1, U7.8 (SW)
- new net VCCINT_VCC: C23.1, U7.1 (VCC)
- no-connect marks 0 -> 15
