File: keyboard/pcb/plate-left/fw16kb-plate-left.kicad_pcb (KiCad board)
At the start: 2 copper layers, 0 parts

Commit message: keyboard left plate: plate.dxf imported on Edge.Cuts (26 closed loops), 1.2 mm; DRC clean
Co-Authored-By: Claude Opus 5.5 (1M context) <noreply@anthropic.com>
Claude-Session: https://claude.ai/code/session_019QA2U79cSHCaAaMe6Km575
Other:
- board outline added: 123.3 x 87.2 mm
